Commit message: allow naming sonar parameters

File: gtri_based_fls_gazebo/urdf/gtri_based_fls.xacro (robot description, xacro)
@@ -1,5 +1,11 @@
 <?xml version="1.0"?>
 <robot xmlns:xacro="http://www.ros.org/wiki/xacro">
-  <xacro:macro name="gtri_based_fls">
+  <xacro:macro name="gtri_based_fls" params="namespace suffix parent_link topic *origin">
+    <!-- joint to Sonar link -->
+    <joint name="${namespace}_gtri_based_fls${suffix}_joint" type="fixed">
+      <parent link="${parent_link}" />
+      <child link="${namespace}/gtri_based_fls${suffix}_link" />
+      <xacro:insert_block name="origin" />
+    </joint>
   <!--
       raycount: number of actual rays used in gazebo
@@ -7,5 +13,5 @@
       If rayCount is less than rangeCount, it will interpolate.
   -->
-    <link name="gtri_based_fls">
+    <link name="${namespace}/gtri_based_fls${suffix}_link">
       <inertial>
         <origin xyz="0 0 0" rpy="0 0 0"/>
@@ -26,7 +32,6 @@
       </visual>
     </link>
-  <gazebo reference="gtri_based_fls">
+  <gazebo reference="${namespace}/gtri_based_fls${suffix}_link">
     <selfCollide>false</selfCollide>
-    <turnGravityOff>true</turnGravityOff>
     <sensor type="ray" name="ray_sensor">
       <always_on>true</always_on>
@@ -62,9 +67,9 @@
           <alwaysOn>true</alwaysOn>
           <updateRate>30.0</updateRate>
-          <linkName>sonar_link</linkName>
-          <frameName>sonar_link</frameName>
-          <cloudTopicName>sonar_cloud</cloudTopicName>
-          <imageTopicName>sonar_image</imageTopicName>
-          <imageCameraInfoTopicName>sonar_image_camera_info</imageCameraInfoTopicName>
+          <linkName>${namespace}/gtri_based_fls${suffix}_link</linkName>
+          <frameName>${namespace}/gtri_based_fls${suffix}_link</frameName>
+          <cloudTopicName>${topic}${suffix}_cloud</cloudTopicName>
+          <imageTopicName>${topic}${suffix}_image</imageTopicName>
+          <imageCameraInfoTopicName>${topic}${suffix}_image_camera_info</imageCameraInfoTopicName>
           <horizontalMinAngle>-0.39269875</horizontalMinAngle>
           <horizontalMaxAngle>0.39269875</horizontalMaxAngle>

File: gtri_based_fls_gazebo/urdf/standalone_gtri_based_fls_robot.xacro (robot description, xacro)
@@ -3,10 +3,11 @@
        xmlns:xacro="http://www.ros.org/wiki/xacro">
   <xacro:include filename="$(find gtri_based_fls)/urdf/gtri_based_fls.xacro" />
-  <xacro:gtri_based_fls/>
   <link name="world"/>
-  <joint name="fixed_gtri_based_fls" type="fixed">
-    <parent link="world"/>
-    <child link="gtri_based_fls"/>
+  <xacro:gtri_based_fls
+            namespace="standalone_gtri_based_fls_robot"
+            suffix="1"
+            parent_link="world"
+            topic="gtri_based_fls">
     <origin xyz="2.1 1.0 1.0" rpy="0 0 1.5709"/>
-  </joint>
+  </xacro:gtri_based_fls>
 </robot>
